File: DroneFlightController/DroneFlightController.kicad_sch (KiCad schematic)
At the start: 24 parts, among them J1 USB_C_Receptacle_USB2.0_14P, U1 STM32F405RGTx, U2 AMS1117-3.3, U3 LSM6DSK320X, U4 AMS1117-3.3

Commit message: add DPS368XTSA1 barometer to MCU I2C1
Parts:
- removed C16, C17: 100nF, symbol Device:C
- removed U3: LSM6DSK320X, symbol DroneProjectLib:LSM6DSK320X
- added C18, C19, C20, C21: 100nF, symbol Device:C
- added R3, R4: 10k, symbol Device:R
- added U5: LSM6DSK320X, symbol DroneProjectLib:LSM6DSK320X
- added U6: (no value), symbol DroneProjectLib:DPS368XTSA1
Connections:
- net GND: now also C18.2, C19.2, C20.2, C21.2, U5.2 (SDx), U5.3 (SCx), U5.6 (GND), U5.7 (GND), U6.1 (GND), U6.7 (GND)
- net IMU_INT1: now also U5.4 (INT1)
- net IMU_INT2: now also U5.9 (INT2)
- net IMU_SPI_CS: now also U5.12 (CS)
- net IMU_SPI_MISO: now also U5.1 (SD0/TA0)
- net IMU_SPI_MOSI: now also U5.14 (SDA)
- net IMU_SPI_SCLK: now also U5.13 (SCL)
- net BAR_I2C_SCK: now reaches U1.58 (PB6)
- net BAR_I2C_SCK: now also R3.1, U6.4 (SCK)
- net BAR_I2C_SDI: now reaches U1.59 (PB7)
- net BAR_I2C_SDI: now also R4.1, U6.3 (SDI)
- new net 3.3V_SENSORS: C18.1, C19.1, C20.1, C21.1, R3.2, R4.2, U5.5 (VDDIO), U5.8 (VDD), U6.6 (VDDIO), U6.8 (VDD)
- no-connect marks 0 -> 2
Other:
- note added: "Barometer"
- note added: "IMU"
